Commit message: feat: add gripper

File: ros2_ws/src/mycobot_description/urdf/mycobot_pro_630/mycobot_pro_630.urdf (robot description, URDF)
Before this commit: robot firefighter, 7 links, 6 joints
Links:
- added link gripper_base, mass 0.07; collision box size=0.065 0.025 0.025; visual mesh filename=file://$(find mycobot_description)/urdf/mycobot_pro_630/gri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
- added link gripper_left1, mass 0.007; collision box size=0.013 0.02 0.015; visual mesh filename=file://$(find mycobot_description)/urdf/mycobot_pro_630/gri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
- added link gripper_left2, mass 0.007; collision box size=0.02 0.02 0.02; visual mesh filename=file://$(find mycobot_description)/urdf/mycobot_pro_630/gri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
- added link gripper_left3, mass 0.007; collision box size=0.01 0.01 0.01; visual mesh filename=file://$(find mycobot_description)/urdf/mycobot_pro_630/gri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
- added link gripper_right1, mass 0.007; collision box size=0.013 0.02 0.015; visual mesh filename=file://$(find mycobot_description)/urdf/mycobot_pro_630/gri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
- added link gripper_right2, mass 0.007; collision box size=0.02 0.02 0.02; visual mesh filename=file://$(find mycobot_description)/urdf/mycobot_pro_630/gri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
- added link gripper_right3, mass 0.007; collision box size=0.01 0.01 0.01; visual mesh filename=file://$(find mycobot_description)/urdf/mycobot_pro_630/gri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
Joints:
- added joint gripper_base_to_gripper_left2: type revolute, parent gripper_base, child gripper_left2, origin xyz=-0.005 0.027 0 rpy=0 0 0, axis 0 0 1, limit lower=-0.8 upper=0.5 effort=5.0 velocity=2.792527, mimic joint=gripper_controller multiplier=1.0 offset=0
- added joint gripper_base_to_gripper_right2: type revolute, parent gripper_base, child gripper_right2, origin xyz=0.005 0.027 0 rpy=0 0 0, axis 0 0 1, limit lower=-0.5 upper=0.8 effort=5.0 velocity=2.792527, mimic joint=gripper_controller multiplier=-1.0 offset=0
- added joint gripper_base_to_gripper_right3: type revolute, parent gripper_base, child gripper_right3, origin xyz=0.012 0.005 0 rpy=0 0 0, axis 0 0 1, limit lower=-0.15 upper=0.7 effort=5.0 velocity=2.792527, mimic joint=gripper_controller multiplier=-1.0 offset=0
- added joint gripper_controller: type revolute, parent gripper_base, child gripper_left3, origin xyz=-0.012 0.005 0 rpy=0 0 0, axis 0 0 1, limit lower=-0.7 upper=0.15 effort=5.0 velocity=2.792527
- added joint gripper_left3_to_gripper_left1: type revolute, parent gripper_left3, child gripper_left1, origin xyz=-0.027 0.016 0 rpy=0 0 0, axis 0 0 1, limit lower=-0.5 upper=0.5 effort=5.0 velocity=2.792527, mimic joint=gripper_controller multiplier=-1.0 offset=0
- added joint gripper_right3_to_gripper_right1: type revolute, parent gripper_right3, child gripper_right1, origin xyz=0.027 0.016 0 rpy=0 0 0, axis 0 0 1, limit lower=-0.5 upper=0.5 effort=5.0 velocity=2.792527, mimic joint=gripper_controller multiplier=1.0 offset=0
- added joint link6_to_gripper_base: type fixed, parent link6, child gripper_base, origin xyz=-0.03 0 0 rpy=1.5707 1.5707 3.142
