Commit message: chore: reference COLLADA files via package share

File: ros2_ws/src/robot_arm/description/models/kuka-lwr-4plus/model.urdf (robot description, URDF)
Before this commit: robot kuka-lwr, 9 links, 8 joints
Links:
- link lwr_arm_1_link: geometry collision mesh filename=file://$(find robot_arm)/description/models/kuka-lwr-4plus/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 scale=1.0 1.0 1.0; visual mesh filename=file://$(find robot_arm)/description/models/kuka-lwr-4plus/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 scale=100 100 100
- link lwr_arm_2_link: geometry collision mesh filename=file://$(find robot_arm)/description/models/kuka-lwr-4plus/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 scale=1.0 1.0 1.0; visual mesh filename=file://$(find robot_arm)/description/models/kuka-lwr-4plus/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 scale=100 100 100
- link lwr_arm_3_link: geometry collision mesh filename=file://$(find robot_arm)/description/models/kuka-lwr-4plus/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 scale=1.0 1.0 1.0; visual mesh filename=file://$(find robot_arm)/description/models/kuka-lwr-4plus/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 scale=100 100 100
- link lwr_arm_4_link: geometry collision mesh filename=file://$(find robot_arm)/description/models/kuka-lwr-4plus/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 scale=1.0 1.0 1.0; visual mesh filename=file://$(find robot_arm)/description/models/kuka-lwr-4plus/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 scale=100 100 100
- link lwr_arm_5_link: geometry collision mesh filename=file://$(find robot_arm)/description/models/kuka-lwr-4plus/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 scale=1.0 1.0 1.0; visual mesh filename=file://$(find robot_arm)/description/models/kuka-lwr-4plus/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 scale=100 100 100
- link lwr_arm_6_link: geometry collision mesh filename=file://$(find robot_arm)/description/models/kuka-lwr-4plus/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 scale=1.0 1.0 1.0; visual mesh filename=file://$(find robot_arm)/description/models/kuka-lwr-4plus/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 scale=100 100 100
- link lwr_arm_7_link: geometry collision mesh filename=file://$(find robot_arm)/description/models/kuka-lwr-4plus/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 scale=100 100 100; visual mesh filename=file://$(find robot_arm)/description/models/kuka-lwr-4plus/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 scale=100 100 100
- link lwr_arm_base_link: geometry collision mesh filename=file://$(find robot_arm)/description/models/kuka-lwr-4plus/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 scale=0.9 0.9 0.9; visual mesh filename=file://$(find robot_arm)/description/models/kuka-lwr-4plus/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 scale=100 100 100
