Commit message: feat(environment_gazebo): model visualization

File: ros2_ws/src/mycobot_description/urdf/model.urdf.xacro (robot description, xacro)
@@ -5,5 +5,5 @@
     <visual>
       <geometry>
-       <mesh filename="file://$(find mycobot_description)/urdf/mycobot_pro_630/base.dae"/>
+       <mesh filename="file://$(find mycobot_description)/urdf/base.dae"/>
       </geometry>
     <origin xyz = "0 0 0 " rpy = " 1.5707 0 0"/>
@@ -11,5 +11,5 @@
     <collision>
     <geometry>
-       <mesh filename="file://$(find mycobot_description)/urdf/mycobot_pro_630/base.dae"/>
+       <mesh filename="file://$(find mycobot_description)/urdf/base.dae"/>
       </geometry>
     <origin xyz = "0 0 0 " rpy = " 1.5707 0 0"/>
@@ -19,5 +19,5 @@
     <visual>
       <geometry>
-       <mesh filename="file://$(find mycobot_description)/urdf/mycobot_pro_630/link1.dae"/>
+       <mesh filename="file://$(find mycobot_description)/urdf/link1.dae"/>
       </geometry>
     <origin xyz = "0 0 -0.06 " rpy = "0 0 3.1415926"/>
@@ -25,5 +25,5 @@
      <collision>
       <geometry>
-       <mesh filename="file://$(find mycobot_description)/urdf/mycobot_pro_630/link1.dae"/>
+       <mesh filename="file://$(find mycobot_description)/urdf/link1.dae"/>
       </geometry>
     <origin xyz = "0 0 -0.06 " rpy = " 0 0 3.1415926"/>
@@ -33,5 +33,5 @@
     <visual>
       <geometry>
-       <mesh filename="file://$(find mycobot_description)/urdf/mycobot_pro_630/link2.dae"/>
+       <mesh filename="file://$(find mycobot_description)/urdf/link2.dae"/>
       </geometry>
     <origin xyz = "0 0 -0.0446 " rpy = " 0 -1.5707 -1.5707"/>
@@ -39,5 +39,5 @@
      <collision>
      <geometry>
-       <mesh filename="file://$(find mycobot_description)/urdf/mycobot_pro_630/link2.dae"/>
+       <mesh filename="file://$(find mycobot_description)/urdf/link2.dae"/>
       </geometry>
     <origin xyz = "0 0 -0.0446 " rpy = " 0 -1.5707 -1.5707"/>
@@ -47,5 +47,5 @@
     <visual>
       <geometry>
-       <mesh filename="file://$(find mycobot_description)/urdf/mycobot_pro_630/link3.dae"/>
+       <mesh filename="file://$(find mycobot_description)/urdf/link3.dae"/>
       </geometry>
     <origin xyz = "0 0 -0.0444 " rpy = " 0 1.5707 -1.5707"/>
@@ -53,5 +53,5 @@
      <collision>
       <geometry>
-       <mesh filename="file://$(find mycobot_description)/urdf/mycobot_pro_630/link3.dae"/>
+       <mesh filename="file://$(find mycobot_description)/urdf/link3.dae"/>
       </geometry>
     <origin xyz = "0 0 -0.0444 " rpy = "0 1.5707 -1.5707"/>
@@ -61,5 +61,5 @@
     <visual>
       <geometry>
-       <mesh filename="file://$(find mycobot_description)/urdf/mycobot_pro_630/link4.dae"/>
+       <mesh filename="file://$(find mycobot_description)/urdf/link4.dae"/>
       </geometry>
     <origin xyz = "0 0 0.041 " rpy = " -1.5707 0 1.5707"/>
@@ -67,5 +67,5 @@
      <collision>
      <geometry>
-       <mesh filename="file://$(find mycobot_description)/urdf/mycobot_pro_630/link4.dae"/>
+       <mesh filename="file://$(find mycobot_description)/urdf/link4.dae"/>
       </geometry>
     <origin xyz = "0 0 0.041 " rpy = " -1.5707 0 1.5707"/>
@@ -75,5 +75,5 @@
     <visual>
       <geometry>
-       <mesh filename="file://$(find mycobot_description)/urdf/mycobot_pro_630/link5.dae"/>
+       <mesh filename="file://$(find mycobot_description)/urdf/link5.dae"/>
       </geometry>
     <origin xyz = "-0.043 0  0 " rpy = " 0  -1.5707 3.1415926"/>
@@ -81,5 +81,5 @@
      <collision>
       <geometry>
-       <mesh filename="file://$(find mycobot_description)/urdf/mycobot_pro_630/link5.dae"/>
+       <mesh filename="file://$(find mycobot_description)/urdf/link5.dae"/>
       </geometry>
     <origin xyz = "-0.043 0  0 " rpy = " 0  -1.5707 3.1415926"/>
@@ -89,5 +89,5 @@
     <visual>
       <geometry>
-       <mesh filename="file://$(find mycobot_description)/urdf/mycobot_pro_630/link6.dae"/>
+       <mesh filename="file://$(find mycobot_description)/urdf/link6.dae"/>
       </geometry>
       <!-- <material name = "grey">
@@ -98,5 +98,5 @@
      <collision>
      <geometry>
-       <mesh filename="file://$(find mycobot_description)/urdf/mycobot_pro_630/link6.dae"/>
+       <mesh filename="file://$(find mycobot_description)/urdf/link6.dae"/>
       </geometry>
       <!-- <material name = "grey">
@@ -118,5 +118,5 @@
 		<visual>
 		  	<geometry>
-				<mesh filename="file://$(find mycobot_description)/urdf/mycobot_pro_630/gripper_base.dae"/>
+				<mesh filename="file://$(find mycobot_description)/urdf/gripper_base.dae"/>
 		  	</geometry>
 		  	<origin xyz = "0.0 0.0 -0.012" rpy = "0 0 0"/>
@@ -140,5 +140,5 @@
 		<visual>
 		  	<geometry>
-		  		<mesh filename="file://$(find mycobot_description)/urdf/mycobot_pro_630/gripper_left1.dae"/>
+		  		<mesh filename="file://$(find mycobot_description)/urdf/gripper_left1.dae"/>
 		  	</geometry>
 			<origin xyz = "0.039 -0.0133 -0.012 " rpy = " 0 0 0"/>
@@ -162,5 +162,5 @@
 		<visual>
 		  	<geometry>
-		   		<mesh filename="file://$(find mycobot_description)/urdf/mycobot_pro_630/gripper_left2.dae"/>
+		   		<mesh filename="file://$(find mycobot_description)/urdf/gripper_left2.dae"/>
 		  	</geometry>
 			<origin xyz = "0.005 -0.0195 -0.012 " rpy = " 0 0 0"/>
@@ -184,5 +184,5 @@
 		<visual>
 		  	<geometry>
-		   		<mesh filename="file://$(find mycobot_description)/urdf/mycobot_pro_630/gripper_left3.dae"/>
+		   		<mesh filename="file://$(find mycobot_description)/urdf/gripper_left3.dae"/>
 		  	</geometry>
 		<origin xyz = "0.012 0.0025 -0.012 " rpy = " 0 0 0"/>
@@ -206,5 +206,5 @@
 		<visual>
 			<geometry>
-		   		<mesh filename="file://$(find mycobot_description)/urdf/mycobot_pro_630/gripper_right1.dae"/>
+		   		<mesh filename="file://$(find mycobot_description)/urdf/gripper_right1.dae"/>
 		  	</geometry>
 			<origin xyz = "-0.039 -0.0133 -0.012 " rpy = " 0 0 0"/>
@@ -228,5 +228,5 @@
 		<visual>
 			<geometry>
-		   		<mesh filename="file://$(find mycobot_description)/urdf/mycobot_pro_630/gripper_right2.dae"/>
+		   		<mesh filename="file://$(find mycobot_description)/urdf/gripper_right2.dae"/>
 		 	</geometry>
 			<origin xyz = "-0.005 -0.0195 -0.012 " rpy = " 0 0 0"/>
@@ -250,5 +250,5 @@
 		<visual>
 			<geometry>
-		   		<mesh filename="file://$(find mycobot_description)/urdf/mycobot_pro_630/gripper_right3.dae"/>
+		   		<mesh filename="file://$(find mycobot_description)/urdf/gripper_right3.dae"/>
 			</geometry>
 			<origin xyz = "-0.012 0.0025 -0.012 " rpy = " 0 0 0"/>
